Commit message: Rename ROS package turtlebot3_gazebo -> multimodal_robot_autonomy
Completes the package rename across the build and simulation tree:
- CMakeLists project() name, so install() targets share/multimodal_robot_autonomy
- include/turtlebot3_gazebo -> include/multimodal_robot_autonomy, with
  matching #include paths and header guards
- launch files and URDFs now resolve get_package_share_directory(
  'multimodal_robot_autonomy'), which previously pointed at a share dir
  the build never produced

File: urdf/turtlebot3_burger.urdf (robot description, URDF)
Before this commit: robot turtlebot3_burger, 7 links, 6 joints
Links:
- link base_link: geometry collision box size=0.140 0.140 0.143; visual mesh filename=package://multimodal_robot_autonomy/models/turtlebot3_commo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 scale=0.001 0.001 0.001
- link base_scan: geometry collision cylinder length=0.0315 radius=0.055; visual mesh filename=package://multimodal_robot_autonomy/models/turtlebot3_commo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 scale=0.001 0.001 0.001
- link wheel_left_link: geometry collision cylinder length=0.018 radius=0.033; visual mesh filename=package://multimodal_robot_autonomy/models/turtlebot3_commo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 scale=0.001 0.001 0.001
- link wheel_right_link: geometry collision cylinder length=0.018 radius=0.033; visual mesh filename=package://multimodal_robot_autonomy/models/turtlebot3_commo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 scale=0.001 0.001 0.001

File: urdf/turtlebot3_burger_cam.urdf (robot description, URDF)
Before this commit: robot turtlebot3_burger_cam, 10 links, 9 joints
Links:
- link base_link: geometry collision box size=0.140 0.140 0.143; visual mesh filename=package://multimodal_robot_autonomy/models/turtlebot3_commo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 scale=0.001 0.001 0.001
- link base_scan: geometry collision cylinder length=0.0315 radius=0.055; visual mesh filename=package://multimodal_robot_autonomy/models/turtlebot3_commo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 scale=0.001 0.001 0.001
- link wheel_left_link: geometry collision cylinder length=0.018 radius=0.033; visual mesh filename=package://multimodal_robot_autonomy/models/turtlebot3_commo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 scale=0.001 0.001 0.001
- link wheel_right_link: geometry collision cylinder length=0.018 radius=0.033; visual mesh filename=package://multimodal_robot_autonomy/models/turtlebot3_commo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 scale=0.001 0.001 0.001

File: urdf/turtlebot3_waffle.urdf (robot description, URDF)
Before this commit: robot turtlebot3_waffle, 13 links, 12 joints
Links:
- link base_link: geometry collision box size=0.266 0.266 0.094; visual mesh filename=package://multimodal_robot_autonomy/models/turtlebot3_commo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 scale=0.001 0.001 0.001
- link base_scan: geometry collision cylinder length=0.0315 radius=0.055; visual mesh filename=package://multimodal_robot_autonomy/models/turtlebot3_commo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 scale=0.001 0.001 0.001
- link camera_link: geometry collision box size=0.012 0.132 0.020; visual mesh filename=package://multimodal_robot_autonomy/models/turtlebot3_commo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
- link wheel_left_link: geometry collision cylinder length=0.018 radius=0.033; visual mesh filename=package://multimodal_robot_autonomy/models/turtlebot3_commo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 scale=0.001 0.001 0.001
- link wheel_right_link: geometry collision cylinder length=0.018 radius=0.033; visual mesh filename=package://multimodal_robot_autonomy/models/turtlebot3_commo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 scale=0.001 0.001 0.001

File: urdf/turtlebot3_waffle_pi.urdf (robot description, URDF)
Before this commit: robot turtlebot3_waffle_pi, 11 links, 10 joints
Links:
- link base_link: geometry collision box size=0.266 0.266 0.094; visual mesh filename=package://multimodal_robot_autonomy/models/turtlebot3_commo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 scale=0.001 0.001 0.001
- link base_scan: geometry collision cylinder length=0.0315 radius=0.055; visual mesh filename=package://multimodal_robot_autonomy/models/turtlebot3_commo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 scale=0.001 0.001 0.001
- link wheel_left_link: geometry collision cylinder length=0.018 radius=0.033; visual mesh filename=package://multimodal_robot_autonomy/models/turtlebot3_commo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 scale=0.001 0.001 0.001
- link wheel_right_link: geometry collision cylinder length=0.018 radius=0.033; visual mesh filename=package://multimodal_robot_autonomy/models/turtlebot3_commo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 scale=0.001 0.001 0.001
