Commit message: Fix empty world regression and unblock the ROMR camera
Two problems, both visible as soon as the sim was actually looked at:

1. The world was empty. Vendoring pulled in romr_simulation's
   small_house.world, which is a 14-line stub (sun + ground plane only) --
   the real house is the AWS world, 837 lines and 89 model includes. Pointing
   gazebo_romr.launch.py at the package copy "for self-containment" therefore
   swapped the house for bare ground; self-containment was never possible
   here anyway since the geometry lives in the AWS models dir. The world path
   is external again, and the stub is renamed worlds/romr_empty.world so it
   stops shadowing the real name.
   Verified: 88 models in the world, was 2.

2. The camera saw nothing but its own hull. camerad435i_link sat at
   x=-0.20718 while base_link spans x=[-0.229, +0.271], leaving 0.48 m of
   robot directly in front of the lens; the sensor has no <pose> override, so
   it looks along +X (forward, confirmed by odometry) from inside the body.
   Captured frames were uniform -- 3 unique colours, std 0.54, and unchanged
   by rotating in place, ruling out a nearby wall. Remounted on the front
   face at x=0.28, centred.
   Verified: 7739 unique colours, std 62.19, house interior in frame.

File: urdf/romr.urdf.xacro (robot description, xacro)
@@ -204,5 +204,12 @@
   </link>
   <joint name="camerad435i_joint" type="fixed">
-    <origin xyz="-0.20718 -0.08268 0.17016" rpy="0 0 0" />
+    <!--
+      Mounted on the front face of the chassis. The upstream pose put this at
+      x=-0.20718, inside the body (base_link spans x=[-0.229, +0.271]), so the
+      camera rendered nothing but the inside of its own hull. base_link +X is
+      forward, confirmed by odometry, and the sensor has no <pose> override, so
+      it looks straight down the length of the robot from wherever it sits.
+    -->
+    <origin xyz="0.28 0 0.17016" rpy="0 0 0" />
     <parent  link="base_link" />
     <child link="camerad435i_link" />

Commit message: Mount the camera flush to the basket rim instead of floating
The previous fix put the camera at x=0.28, derived from base_link's overall
bounding box max (x=+0.271) -- but that maximum comes from the caster mount
low down, not from the cart body at camera height. At z~0.17 on the centreline
the hull actually ends at x=-0.185, because that height is the open gap between
the lower deck and the basket, so the camera hung visibly detached in front of
the robot.

Mounted on the basket rim's front face instead: x=0.235, z=0.21, which sits
4mm proud of the hull surface at that height (x=+0.2308 for z in 0.20..0.25).

Verified: TF base_link->camerad435i_link = [0.235, 0.000, 0.210], and captured
frames still show the house interior with no chassis in view (3974 colours,
std 42.8).

File: urdf/romr.urdf.xacro (robot description, xacro)
@@ -205,11 +205,17 @@
   <joint name="camerad435i_joint" type="fixed">
     <!--
-      Mounted on the front face of the chassis. The upstream pose put this at
-      x=-0.20718, inside the body (base_link spans x=[-0.229, +0.271]), so the
-      camera rendered nothing but the inside of its own hull. base_link +X is
-      forward, confirmed by odometry, and the sensor has no <pose> override, so
-      it looks straight down the length of the robot from wherever it sits.
+      Mounted flush on the front face of the basket rim, which is the hull's
+      forward-most surface at this height (x=+0.2308 for z in 0.20..0.25).
+      Do not derive this from the mesh's overall bounding box: at the camera's
+      own height on the centreline the hull ends at x=-0.185, because z~0.17 is
+      the open gap between the lower deck and the basket, so a pose picked from
+      the global max (x=+0.271, which comes from the caster mount low down)
+      leaves the camera floating unattached in front of the robot.
+      The upstream pose put this at x=-0.20718, inside the body, so the camera
+      rendered nothing but the inside of its own hull. base_link +X is forward,
+      confirmed by odometry, and the sensor has no <pose> override, so it looks
+      straight down the length of the robot from wherever it sits.
     -->
-    <origin xyz="0.28 0 0.17016" rpy="0 0 0" />
+    <origin xyz="0.235 0 0.21" rpy="0 0 0" />
     <parent  link="base_link" />
     <child link="camerad435i_link" />

Commit message: Fix ROMR's drivetrain so it can actually drive
Mapping runs kept wedging the robot (48 stuck events in 5 minutes, actual
velocity ~0 while cmd_vel commanded a turn). Four separate defects:

- casterwheel_joint is FIXED, so the caster is a dragging skid, but it had
  mu=1.0 against drive wheels at mu=1000. Set to frictionless with slip, the
  standard way to model a fixed caster.
- The caster sat 12.7mm too low: its underside was at -0.1587 while the wheels
  contact at -0.146, so the robot rested nose-down with the drive wheels
  partly unloaded. Raised to -0.0948 = wheel contact plane + caster radius.
- wheel_separation and wheel_diameter are now calibrated against measured
  response rather than nominal values. Note the URDF joint spacing (0.370) is
  NOT the effective contact separation: configuring it made turns 26% fast.
  Effective value is 0.2937, so upstream's 0.30 was very nearly right.
- worlds/romr_empty.world pulled its floor from model://ground_plane, which
  resolves against Gazebo's online model database and is unreachable here, so
  the world loaded with no floor. Ground plane and light are now inline.

Verified on flat ground with collision geometry loaded: robot rests at
z=0.1415 and tracks commands within 4% --
  v 0.25 -> 0.260 | w +0.80 -> +0.824 | w -0.80 -> -0.825 | arc 0.20/0.50 -> 0.205/0.518
Previously: v 0.25 -> 0.128, and left turns did not execute at all.

File: urdf/romr.urdf.xacro (robot description, xacro)
@@ -123,5 +123,14 @@
   </link>
   <joint name="casterwheel_joint" type="fixed">
-    <origin xyz="0.25029 -0.01098 -0.1075" rpy="0 0 0" />
+    <!--
+      z was -0.1075, which put the caster's underside at -0.1587 while the
+      drive wheels contact at -0.146 (joint z=-0.063 minus measured wheel
+      radius 0.083). The robot therefore rested nose-down on the caster with
+      the drive wheels partly unloaded, giving poor traction, veer on straight
+      commands and a turn that only worked in one direction.
+      -0.0948 = wheel contact plane (-0.146) + caster radius (0.0512), so the
+      caster just touches the same ground plane as the wheels.
+    -->
+    <origin xyz="0.25029 -0.01098 -0.0948" rpy="0 0 0" />
     <parent link="base_link" />
     <child link="casterwheel_link" />

Commit message: Raise the lidar above the cart and re-slice the map to match
The lidar sat at z=+0.12332 while the base_link mesh spans z=-0.091..+0.287,
so the scan plane cut through ROMR's own cart: 56 of 720 beams returned hits
on the robot itself at 0.167..0.311 m, ringing it with phantom obstacles.

The first attempt raised the sensor's min range to 0.33 to filter the
self-hits. That worked, but traded one failure for another: obstacles vanished
from the scan once they came within 0.33 m, so the local costmap cleared them
and the controller drove into contact. A navigation run ended with the robot
at 0.20 m clearance, inside lethal space for a 0.33 m radius, and the planner
then refused every goal because the START was blocked.

Raising lidar_joint to z=0.30, just above the basket rim, fixes it properly:
clear 360 view, and the sensor keeps its true 0.15 m minimum range.

The map is regenerated to match, sliced at the new lidar height 0.4415 m
(base rests at 0.1415, plus 0.30). 1241 cells differ from the 0.265 slice,
mostly low furniture that no longer intersects the beam plane.

File: urdf/romr.urdf.xacro (robot description, xacro)
@@ -159,5 +159,13 @@
   </link>
   <joint name="lidar_joint" type="fixed">
-    <origin xyz="0.00082049 0.00875 0.12332" rpy="0 0 0" />
+    <!--
+      z was 0.12332, which put the scan plane INSIDE the cart: the base_link
+      mesh spans z -0.091..+0.287, so 56 of 720 beams hit the robot itself.
+      Raised to 0.30, just above the basket rim, so the scanner has a clear
+      360 view and can keep its true 0.15 m minimum range. Blinding the sensor
+      below 0.33 instead let obstacles vanish once they got close, and the
+      controller then drove into them.
+    -->
+    <origin xyz="0.00082049 0.00875 0.30" rpy="0 0 0" />
     <parent link="base_link" />
     <child link="lidar_link" />

Commit message: Give ROMR a rear caster so it stops tipping over backwards
ROMR shipped with a single caster at the FRONT (x=+0.250). The rearmost ground
contact was therefore the wheel axle at x=-0.124, with the centre of mass only
0.0865 m ahead of it -- a 24.1 degree rear tipping margin on a robot whose CoM
sits 0.193 m above the floor.

Measured in a purpose-built rig (flat ground, a 0.22 m door-frame post offset
to strike one side, ground truth from gazebo_ros_state because wheel odometry
is synthesised in 2-D and reports the robot upright even when it is on its
side):

  baseline      0.22 m/s   pitch 40.5 deg   upright
  baseline      0.35 m/s   pitch 50.2 deg   TIPPED   (roll only 7.4 deg)

The low roll is the tell: it was not rolling sideways, it pivoted nose-up about
the wheel axle and went over backwards. A full-width kerb is struck
symmetrically and simply climbed, which is why this only showed up against
door frames.

A second caster at x=-0.20 -- inside the body, which reaches -0.229, and at the
same z so both touch the wheels' ground plane -- extends the support polygon
rearward and raises the margin to 40.1 degrees:

  rear caster   0.22 m/s   pitch  3.8 deg   upright
  rear caster   0.35 m/s   pitch 10.5 deg   upright
  rear caster   0.45 m/s   pitch 10.6 deg   upright

With the cause fixed, the controller limits lowered as a stopgap are restored:
max_vel_x and max_speed_xy back to 0.35, acc_lim_x 1.5, acc_lim_theta 2.0.

File: urdf/romr.urdf.xacro (robot description, xacro)
@@ -135,4 +135,42 @@
     <parent link="base_link" />
     <child link="casterwheel_link" />
+    <axis xyz="0 0 0" />
+  </joint>
+  <!--
+    Rear caster. ROMR shipped with a single caster at the FRONT (x=+0.250), so
+    the rearmost ground contact was the wheel axle at x=-0.124 and the centre of
+    mass sat only 0.0865 m ahead of it: a 24.1 deg rear tipping margin. Striking
+    a door frame asymmetrically pivoted the robot nose-up about that axle and
+    over; measured 50.2 deg of pitch at 0.35 m/s in the tip rig, with only
+    7.4 deg of roll, so it went over backwards rather than sideways.
+    Placing a second caster at x=-0.20 (inside the body, which reaches -0.229)
+    extends the support polygon rearward and raises that margin to 40.0 deg.
+    z matches the front caster so both touch the wheels' ground plane.
+  -->
+  <link name="rearcaster_link">
+    <inertial>
+      <origin xyz="-0.0032546 0.0053327 0.013127" rpy="0 0 0" />
+      <mass value="0.10255" />
+      <inertia ixx="9.4829E-05" ixy="-2.3412E-06" ixz="1.3145E-05" iyy="0.00012884" iyz="8.5135E-07" izz="5.2207E-05" />
+    </inertial>
+    <visual>
+      <origin xyz="0 0 0" rpy="0 0 0" />
+      <geometry>
+        <mesh filename="package://multimodal_robot_autonomy/meshes/casterwheel.STL" />
+      </geometry>
+      <material name="blue">
+      </material>
+    </visual>
+    <collision>
+      <origin xyz="0 0 0" rpy="0 0 0" />
+      <geometry>
+        <mesh filename="package://multimodal_robot_autonomy/meshes/casterwheel.STL" />
+      </geometry>
+    </collision>
+  </link>
+  <joint name="rearcaster_joint" type="fixed">
+    <origin xyz="-0.20 0.0 -0.0948" rpy="0 0 0" />
+    <parent link="base_link" />
+    <child link="rearcaster_link" />
     <axis xyz="0 0 0" />
   </joint>

Commit message: Fix the drivetrain geometry, and trace the command graph in the UI
The garage goal was not reachable, but neither was anything else: the
planner refused every goal, including a point 0.5 m away, because the
robot's own start cell was lethal. Two model defects behind it.

The caster height was computed from an assumed 0.0512 radius rather than
the mesh. casterwheel.STL actually reaches 0.03791 below its link origin
and the wheels contact at -0.14594 (measured radius 0.08294), so a caster
joint belongs at -0.10803, not -0.0948. That error lifted both casters
13.2 mm clear of the floor: the robot balanced on two wheels, tipped 2 deg
nose-down onto the front caster and dragged it as a skid.

max_wheel_acceleration was 1.0 rad/s^2 = 0.081 m/s^2, while DWB simulates
every trajectory against acc_lim_x 1.5 -- an 18x mismatch, which is what
produced "No valid trajectories out of 419!". Now 18.5 = 1.5 / 0.08135.

Together these took the robot from 10-14% of commanded speed to 90%.

The place poses were never at fault: garage is x=3.20 y=-5.50 yaw=-1.57 at
every commit of the original repo including the first, and the transform
into world coordinates is exact for all seven places.

The command graph now records a step per node -- when it ran, how long it
took, and which branch it took and why -- exposed as `trace` alongside the
existing node trail. The new Reasoning page draws the graph and lights up
the route a run actually took, so a recovery retry is visible as a loop
rather than inferred from a log.

File: urdf/romr.urdf.xacro (robot description, xacro)
@@ -124,13 +124,19 @@
   <joint name="casterwheel_joint" type="fixed">
     <!--
-      z was -0.1075, which put the caster's underside at -0.1587 while the
-      drive wheels contact at -0.146 (joint z=-0.063 minus measured wheel
-      radius 0.083). The robot therefore rested nose-down on the caster with
-      the drive wheels partly unloaded, giving poor traction, veer on straight
-      commands and a turn that only worked in one direction.
-      -0.0948 = wheel contact plane (-0.146) + caster radius (0.0512), so the
-      caster just touches the same ground plane as the wheels.
+      Ground contact heights, all measured from the mesh files rather than
+      assumed:
+        leftwheel.STL / rightwheel.STL  radius 0.08294  (bbox 0.16588 across)
+        wheel contact plane            -0.063 - 0.08294 = -0.14594
+        casterwheel.STL                reaches 0.03791 below its link origin
+      so a caster joint sits at -0.14594 + 0.03791 = -0.10803 for its underside
+      to meet the same ground plane as the wheels.
+      This was briefly -0.0948, computed from an assumed caster radius of
+      0.0512 instead of the mesh's actual 0.03791 drop. That lifted both
+      casters 13.2 mm clear of the floor, so the robot balanced on the two
+      drive wheels alone and tipped nose-down 2 deg onto the front caster,
+      dragging it as a skid: it reached only 14% of commanded speed
+      (0.021 m/s against 0.15 m/s commanded) and nav2 aborted continually.
     -->
-    <origin xyz="0.25029 -0.01098 -0.0948" rpy="0 0 0" />
+    <origin xyz="0.25029 -0.01098 -0.10803" rpy="0 0 0" />
     <parent link="base_link" />
     <child link="casterwheel_link" />
@@ -146,5 +152,6 @@
     Placing a second caster at x=-0.20 (inside the body, which reaches -0.229)
     extends the support polygon rearward and raises that margin to 40.0 deg.
-    z matches the front caster so both touch the wheels' ground plane.
+    z matches the front caster so both touch the wheels' ground plane; see the
+    derivation on casterwheel_joint.
   -->
   <link name="rearcaster_link">
@@ -170,5 +177,5 @@
   </link>
   <joint name="rearcaster_joint" type="fixed">
-    <origin xyz="-0.20 0.0 -0.0948" rpy="0 0 0" />
+    <origin xyz="-0.20 0.0 -0.10803" rpy="0 0 0" />
     <parent link="base_link" />
     <child link="rearcaster_link" />

Commit message: Remove the rear caster, and fix the cleanup that never worked
clean.sh ran "pkill -x gzserver gzclient robot_state_publisher". pkill
takes a single pattern and rejects the rest, so only gzserver was ever
killed. Twenty-two robot_state_publishers had accumulated, the oldest
6.4 hours old, each publishing its own /robot_description and TF. Every
measurement taken today was against that. One pattern per pkill now.

The rear caster is gone. ROMR has one caster, at the front; the second
was added at x=-0.20 to stop the robot tipping backwards, but two wheels
plus two casters is four ground contacts on a rigid body, which is
statically over-constrained. The tipping it addressed was compounded by
two defects since fixed, so the fourth contact was probably never the
right remedy. Rear tipping margin returns to 24.1 degrees; if tipping
recurs, widen the wheelbase or move mass forward rather than adding a
fourth contact.

check_xml.sh rejects "--" inside an XML comment before xacro sees it.
That has broken the build three times, always an em-dash written as two
hyphens, and xacro only reports "not well-formed (invalid token)".

File: urdf/romr.urdf.xacro (robot description, xacro)
@@ -144,42 +144,18 @@
   </joint>
   <!--
-    Rear caster. ROMR shipped with a single caster at the FRONT (x=+0.250), so
-    the rearmost ground contact was the wheel axle at x=-0.124 and the centre of
-    mass sat only 0.0865 m ahead of it: a 24.1 deg rear tipping margin. Striking
-    a door frame asymmetrically pivoted the robot nose-up about that axle and
-    over; measured 50.2 deg of pitch at 0.35 m/s in the tip rig, with only
-    7.4 deg of roll, so it went over backwards rather than sideways.
-    Placing a second caster at x=-0.20 (inside the body, which reaches -0.229)
-    extends the support polygon rearward and raises that margin to 40.0 deg.
-    z matches the front caster so both touch the wheels' ground plane; see the
-    derivation on casterwheel_joint.
+    ROMR has one caster, at the FRONT (x=+0.250). A second caster was added at
+    x=-0.20 to extend the support polygon rearward, because the robot tipped
+    backwards when it struck a door frame at 0.35 m/s. It has been removed
+    again: two wheels plus two casters is four contact points on a rigid body,
+    which is statically over-constrained, and the solver's continuous attempt to
+    satisfy all four showed up as the robot creeping while parked.
+    Three contacts are determinate. The tipping it was added to prevent was
+    itself compounded by two defects since fixed — caster height taken from an
+    assumed radius rather than the mesh, and an acceleration limit eighteen
+    times below what the controller assumed — so it is no longer clear the
+    fourth contact was ever the right remedy. Rear tipping margin returns to
+    24.1 deg; if tipping recurs, widen the wheelbase or move mass forward rather
+    than adding a fourth ground contact.
   -->
-  <link name="rearcaster_link">
-    <inertial>
-      <origin xyz="-0.0032546 0.0053327 0.013127" rpy="0 0 0" />
-      <mass value="0.10255" />
-      <inertia ixx="9.4829E-05" ixy="-2.3412E-06" ixz="1.3145E-05" iyy="0.00012884" iyz="8.5135E-07" izz="5.2207E-05" />
-    </inertial>
-    <visual>
-      <origin xyz="0 0 0" rpy="0 0 0" />
-      <geometry>
-        <mesh filename="package://multimodal_robot_autonomy/meshes/casterwheel.STL" />
-      </geometry>
-      <material name="blue">
-      </material>
-    </visual>
-    <collision>
-      <origin xyz="0 0 0" rpy="0 0 0" />
-      <geometry>
-        <mesh filename="package://multimodal_robot_autonomy/meshes/casterwheel.STL" />
-      </geometry>
-    </collision>
-  </link>
-  <joint name="rearcaster_joint" type="fixed">
-    <origin xyz="-0.20 0.0 -0.10803" rpy="0 0 0" />
-    <parent link="base_link" />
-    <child link="rearcaster_link" />
-    <axis xyz="0 0 0" />
-  </joint>
   <link name="lidar_link">
     <inertial>
